File: hardware/Battery power module.kicad_sch (KiCad schematic)
At the start: 15 parts, among them J1 USB_C_Receptacle_PowerOnly_6P, J2 Conn_01x02, U1 BQ24090DGQ

Commit message: Version 1.1: Extending the USB port beyond the board outline and adding a version designation on the PCB
Parts:
- J2: now left out of the parts list
Changed lines of the file:
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@@
 		(unit 1)
 		(exclude_from_sim no)
-		(in_bom yes)
+		(in_bom no)
 		(on_board yes)
 		(dnp no)
